File: CANadapter.sch (KiCad schematic (older format))
At the start: 28 parts, among them P1 CONN_02X06, P2 CONN_01X06, P3 CONN_01X04, P4 CONN_01X06, U1 MCP2515, U2 TLP2361, U3 TLP2361, U4 MCP2551-I/SN, U5 LM7805CT, U6 NKE0305SC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

Commit message: finished routing, improved silk
Parts:
- JP1, JP2: footprint LocalLib:JumperSingleJumbo -> LocalLib:JumperSingleClosed

Commit message: improved silk
Parts:
- JP3, JP4, JP5, JP6: footprint LocalLib:JumperSingleJumbo -> LocalLib:JumperSingle
Changed lines of the file:
@@
 F 0 "JP3" H 7950 2080 50  0000 C CNN
 F 1 "Terminate" H 7960 1940 50  0001 C CNN
-F 2 "LocalLib:JumperSingleJumbo" H 7950 2000 50  0001 C CNN
+F 2 "LocalLib:JumperSingle" H 7950 2000 50  0001 C CNN
 F 3 "" H 7950 2000 50  0000 C CNN
 	1    7950 2000
@@
 F 0 "JP5" H 8150 2080 50  0000 C CNN
 F 1 "Terminate" H 8160 1940 50  0000 C CNN
-F 2 "LocalLib:JumperSingleJumbo" H 8150 2000 50  0001 C CNN
+F 2 "LocalLib:JumperSingle" H 8150 2000 50  0001 C CNN
 F 3 "" H 8150 2000 50  0000 C CNN
 	1    8150 2000
@@
 F 0 "JP4" H 8400 2580 50  0000 C CNN
 F 1 "Filter" H 8410 2440 50  0000 C CNN
-F 2 "LocalLib:JumperSingleJumbo" H 8400 2500 50  0001 C CNN
+F 2 "LocalLib:JumperSingle" H 8400 2500 50  0001 C CNN
 F 3 "" H 8400 2500 50  0000 C CNN
 	1    8400 2500
@@
 F 0 "JP6" H 9700 4230 50  0000 C CNN
 F 1 "Line Power" H 9710 4090 50  0000 C CNN
-F 2 "LocalLib:JumperSingleJumbo" H 9700 4150 50  0001 C CNN
+F 2 "LocalLib:JumperSingle" H 9700 4150 50  0001 C CNN
 F 3 "" H 9700 4150 50  0000 C CNN
 	1    9700 4150
